File: saturn.kicad_sch (KiCad schematic)
At the start: 103 parts, among them J1 Conn_01x04_Pin, J10 Conn_01x04, J11 USB_B_Micro, J12 USB_C_Receptacle_USB2.0, J13 Conn_01x03, J14 Conn_01x04_Pin, J2 PMOD0_FULL, J3 Conn_01x06, J4 Conn_01x06, J6 Conn_01x10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

Commit message: Release v1.0.0
Parts:
- added R19: 10k, Resistor_SMD:R_0402_1005Metric, symbol Device:R
- J13: value Conn_01x03 -> S3B-XH-A-1(LF)(SN); LCSC C493416 -> C163036
- J2: JLCPCB_CORRECTION (none) -> -1.27;6.35;-90
- J3, J4: JLCPCB_CORRECTION (none) -> 0;6.35;-90
- J6: JLCPCB_CORRECTION (none) -> 11.25;0;0
- JP1, JP2, JP3: JLCPCB_CORRECTION (none) -> 0;2.54;90; now in the parts list
- RN1, RN2, RN3, RN4, RN5, RN6: JLCPCB_CORRECTION (none) -> 0;0;90
- U1: JLCPCB_CORRECTION (none) -> 0;9;0
- U2: JLCPCB_CORRECTION (none) -> 0;0;180
- U9: value WS2812B -> XL-2020RGBC-WS2812B; JLCPCB_CORRECTION (none) -> 0;0;180
Connections:
- net +3V3: now also R19.2
- net DISPLAY_CS: now also R19.1
- no-connect marks 6 -> 8
Other:
- moved on the sheet: RN6A

Commit message: Switch to Kicad 10
Parts:
- added unit 3 of RN6
Connections:
- net DISPLAY_CLK: now also RN6.5 (R4.2), RN6.6 (R3.2); no longer RN6.5 (R4.2), RN6.6 (R3.2)
- new net: J6.10 (Pin_10), RN6.3 (R3.1), RN6.4 (R4.1)
Other:
- moved on the sheet: RN6D

Commit message: Fix PMOD ADC pin assignment, tune silkscreen
Parts:
- removed H5, H6, H7: MountingHole, MountingHole:ToolingHole_1.152mm, symbol Mechanical:MountingHole
- J2: value PMOD0_FULL -> PMOD3_FULL
Connections:
- net I2CA_SCL: now also U1.10 (IO17); no longer U1.12 (IO08)
- net I2CA_SDA: now also U1.11 (IO18); no longer U1.17 (IO09)
- net PMOD1_IO1: now also U1.9 (IO16); no longer U1.7 (IO07)
- net PMOD1_IO2: now also U1.8 (IO15); no longer U1.6 (IO06)
- net PMOD2_IO3: now also U1.18 (IO10); no longer U1.24 (IO47)
- net PMOD0_IO1 renamed PMOD3_IO1
- net PMOD0_IO10 renamed PMOD3_IO10
- net PMOD3_IO10: now also U1.6 (IO06); no longer U1.8 (IO15)
- net PMOD0_IO2 renamed PMOD3_IO2
- net PMOD0_IO3 renamed PMOD3_IO3
- net PMOD3_IO3: now also U1.17 (IO09); no longer U1.11 (IO18)
- net PMOD0_IO4 renamed PMOD3_IO4
- net PMOD3_IO4: now also U1.7 (IO07); no longer U1.9 (IO16)
- net PMOD0_IO7 renamed PMOD3_IO7
- net PMOD0_IO8 renamed PMOD3_IO8
- net PMOD3_IO8: now also U1.24 (IO47); no longer U1.18 (IO10)
- net PMOD0_IO9 renamed PMOD3_IO9
- net PMOD3_IO9: now also U1.12 (IO08); no longer U1.10 (IO17)
Other:
- note added: "Analog capable pins: ESP IO01 - IO10 PMOD IO3 and IO4 (and PMOD IO9 and IO10) pins must be within this range"
- note removed: "Analog capable pins: ESP IO01 - IO20 PMOD IO4 (and PMOD IO10) pins must be within this range"

Commit message: Use unipolar TVS diodes, tune switch values
Parts:
- D6, D7, D8, D9: value H3V3LD5B -> PESD3V3L1UB; LCSC C20615817 -> C3001945
- SW2: value EN -> SKRPABE010
- SW3: value BOOT -> SKRPABE010
Changed lines of the file:
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@@
 			)
 		)
-		(property "Value" "BOOT"
+		(property "Value" "SKRPABE010"
 			(at 33.02 203.2 0)
 			(show_name no)
@@
 			)
 		)
-		(property "Value" "H3V3LD5B"
+		(property "Value" "PESD3V3L1UB"
 			(at 52.832 114.808 0)
 			(show_name no)
@@
 			)
 		)
-		(property "Datasheet" "https://jlcpcb.com/api/file/downloadByFileSystemAccessId/8590925461511741440"
+		(property "Datasheet" "https://jlcpcb.com/api/file/downloadByFileSystemAccessId/8590910295219126272"
 			(at 49.53 113.03 0)
 			(hide yes)
@@
 			)
 		)
-		(property "LCSC" "C20615817"
+		(property "LCSC" "C3001945"
 			(at 49.53 114.3 90)
 			(hide yes)
@@
 			)
 		)
-		(property "Value" "H3V3LD5B"
+		(property "Value" "PESD3V3L1UB"
 			(at 41.148 114.808 0)
 			(show_name no)
@@
 			)
 		)
-		(property "Datasheet" "https://jlcpcb.com/api/file/downloadByFileSystemAccessId/8590925461511741440"
+		(property "Datasheet" "https://jlcpcb.com/api/file/downloadByFileSystemAccessId/8590910295219126272"
 			(at 44.45 113.03 0)
 			(hide yes)
@@
 			)
 		)
-		(property "LCSC" "C20615817"
+		(property "LCSC" "C3001945"
 			(at 44.45 114.3 90)
 			(hide yes)
@@
 			)
 		)
-		(property "Value" "H3V3LD5B"
+		(property "Value" "PESD3V3L1UB"
 			(at 67.437 58.928 0)
 			(show_name no)
@@
 			)
 		)
-		(property "Datasheet" "https://jlcpcb.com/api/file/downloadByFileSystemAccessId/8590925461511741440"
+		(property "Datasheet" "https://jlcpcb.com/api/file/downloadByFileSystemAccessId/8590910295219126272"
 			(at 64.135 57.15 0)
 			(hide yes)
@@
 			)
 		)
-		(property "LCSC" "C20615817"
+		(property "LCSC" "C3001945"
 			(at 64.135 58.42 90)
 			(hide yes)
@@
 			)
 		)
-		(property "Value" "H3V3LD5B"
+		(property "Value" "PESD3V3L1UB"
 			(at 55.753 58.928 0)
 			(show_name no)
@@
 			)
 		)
-		(property "Datasheet" "https://jlcpcb.com/api/file/downloadByFileSystemAccessId/8590925461511741440"
+		(property "Datasheet" "https://jlcpcb.com/api/file/downloadByFileSystemAccessId/8590910295219126272"
 			(at 59.055 57.15 0)
 			(hide yes)
@@
 			)
 		)
-		(property "LCSC" "C20615817"
+		(property "LCSC" "C3001945"
 			(at 59.055 58.42 90)
 			(hide yes)
@@
 			)
 		)
-		(property "Value" "EN"
+		(property "Value" "SKRPABE010"
 			(at 33.02 165.1 0)
 			(show_name no)

Commit message: Use SMT PMOD jumper header
Parts:
- JP1, JP2, JP3: footprint Connector_PinHeader_2.54mm:PinHeader_1x03_P2.54mm_Vertical -> PinHeader_jumper:PinHeader_1x03_P2.54mm_Vertical_SMD_Pin1Left_LargePads; JLCPCB_CORRECTION 0;2.54;90 -> (none); LCSC C49257 -> C41417360
Changed lines of the file:
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@@
 			)
 		)
-		(property "Footprint" "Connector_PinHeader_2.54mm:PinHeader_1x03_P2.54mm_Vertical"
+		(property "Footprint" "PinHeader_jumper:PinHeader_1x03_P2.54mm_Vertical_SMD_Pin1Left_LargePads"
 			(at 344.17 85.09 0)
 			(hide yes)
@@
 			)
 		)
-		(property "LCSC" "C49257"
+		(property "LCSC" "C41417360"
 			(at 344.17 85.09 90)
 			(hide yes)
@@
 			)
 		)
-		(property "JLCPCB_CORRECTION" "0;2.54;90"
+		(property "JLCPCB_CORRECTION" ""
 			(at 344.17 85.09 90)
 			(hide yes)
@@
 			)
 		)
-		(property "Footprint" "Connector_PinHeader_2.54mm:PinHeader_1x03_P2.54mm_Vertical"
+		(property "Footprint" "PinHeader_jumper:PinHeader_1x03_P2.54mm_Vertical_SMD_Pin1Left_LargePads"
 			(at 344.17 48.26 0)
 			(hide yes)
@@
 			)
 		)
-		(property "LCSC" "C49257"
+		(property "LCSC" "C41417360"
 			(at 344.17 48.26 90)
 			(hide yes)
@@
 			)
 		)
-		(property "JLCPCB_CORRECTION" "0;2.54;90"
+		(property "JLCPCB_CORRECTION" ""
 			(at 344.17 48.26 90)
 			(hide yes)
@@
 			)
 		)
-		(property "Footprint" "Connector_PinHeader_2.54mm:PinHeader_1x03_P2.54mm_Vertical"
+		(property "Footprint" "PinHeader_jumper:PinHeader_1x03_P2.54mm_Vertical_SMD_Pin1Left_LargePads"
 			(at 262.89 48.26 0)
 			(hide yes)
@@
 			)
 		)
-		(property "LCSC" "C49257"
+		(property "LCSC" "C41417360"
 			(at 262.89 48.26 90)
 			(hide yes)
@@
 			)
 		)
-		(property "JLCPCB_CORRECTION" "0;2.54;90"
+		(property "JLCPCB_CORRECTION" ""
 			(at 262.89 48.26 90)
 			(hide yes)

Commit message: Use SMT JST-XH connectors
Parts:
- J13: value S3B-XH-A-1(LF)(SN) -> ZX-XH2.54-3PWT; footprint Connector_JST:JST_XH_S3B-XH-A-1_1x03_P2.50mm_Horizontal -> JST-XH-SMT:JST-XH-SMD-3Pin; symbol Connector_Generic:Conn_01x03 -> Connector_Generic_MountingPin:Conn_01x03_MountingPin; JLCPCB_CORRECTION 2.54;0;180 -> (none); LCSC C163036 -> C7429672; Price (100ks) 0.0675 -> (none); Price (1ks) 0.0815 -> (none)
- J6: value Conn_01x10 -> ZX-XH2.54-10PWT; footprint Connector_JST:JST_XH_S10B-XH-A-1_1x10_P2.50mm_Horizontal -> JST-XH-SMT:JST-XH-SMD-10Pin; symbol Connector_Generic:Conn_01x10 -> Connector_Generic_MountingPin:Conn_01x10_MountingPin; JLCPCB_CORRECTION 11.25;0;0 -> (none); LCSC C491718 -> C7429679
- JP1, JP2, JP3: JLCPCB_CORRECTION (none) -> 0;0;-90
Connections:
- net GND: now also J13.MP (MountPin), J6.MP (MountPin)
Changed lines of the file:
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@@
 	(wire
 		(pts
+			(xy 394.97 176.53) (xy 394.97 177.8)
+		)
+		(stroke
+			(width 0)
+			(type default)
+		)
+	)
+	(wire
+		(pts
 			(xy 236.22 248.92) (xy 236.22 257.81)
 		)
@@
 	(wire
 		(pts
+			(xy 223.52 31.75) (xy 223.52 26.67)
+		)
+		(stroke
+			(width 0)
+			(type default)
+		)
+	)
+	(wire
+		(pts
+			(xy 229.87 26.67) (xy 229.87 29.21)
+		)
+		(stroke
+			(width 0)
+			(type default)
+		)
+	)
+	(wire
+		(pts
+			(xy 223.52 26.67) (xy 229.87 26.67)
+		)
+		(stroke
+			(width 0)
+			(type default)
+		)
+	)
+	(wire
+		(pts
 			(xy 265.43 229.87) (xy 265.43 233.68)
 		)
@@
 	(wire
 		(pts
+			(xy 389.89 176.53) (xy 394.97 176.53)
+		)
+		(stroke
+			(width 0)
+			(type default)
+		)
+	)
+	(wire
+		(pts
 			(xy 115.57 115.57) (xy 113.03 115.57)
 		)
@@
 	(wire
 		(pts
+			(xy 389.89 182.88) (xy 389.89 176.53)
+		)
+		(stroke
+			(width 0)
+			(type default)
+		)
+	)
+	(wire
+		(pts
 			(xy 267.97 138.43) (xy 287.02 138.43)
 		)
@@
 	(symbol
 		(lib_id "power:GND")
-		(at 373.38 95.25 0)
+		(at 229.87 29.21 0)
+		(mirror y)
 		(unit 1)
 		(body_style 1)
@@
 		(in_pos_files yes)
 		(dnp no)
-		(property "Reference" "#PWR035"
-			(at 373.38 101.6 0)
+		(fields_autoplaced yes)
+		(property "Reference" "#PWR072"
+			(at 229.87 35.56 0)
 			(hide yes)
 			(show_name no)
@@
 		)
 		(property "Value" "GND"
-			(at 373.38 100.33 0)
+			(at 229.87 34.29 0)
 			(show_name no)
 			(do_not_autoplace no)
@@
 		)
 		(property "Footprint" ""
-			(at 373.38 95.25 0)
+			(at 229.87 29.21 0)
 			(hide yes)
 			(show_name no)
@@
 		)
 		(property "Datasheet" ""
-			(at 373.38 95.25 0)
+			(at 229.87 29.21 0)
 			(hide yes)
 			(show_name no)
@@
 		)
 		(property "Description" "Power symbol creates a global label with name \"GND\" , ground"
-			(at 373.38 95.25 0)
+			(at 229.87 29.21 0)
 			(hide yes)
 			(show_name no)
@@
 			(project "saturn"
 				(path "/1437d78f-2672-4553-b786-22c28e887ed9"
-					(reference "#PWR035")
+					(reference "#PWR072")
 					(unit 1)
 				)
@@
 	)
 	(symbol
-		(lib_id "Connector_Generic:Conn_01x03")
-		(at 223.52 39.37 0)
-		(mirror x)
+		(lib_id "power:GND")
+		(at 373.38 95.25 0)
 		(unit 1)
 		(body_style 1)
@@
 		(in_pos_files yes)
 		(dnp no)
-		(fields_autoplaced yes)
-		(property "Reference" "J13"
-			(at 223.52 30.48 0)
+		(property "Reference" "#PWR035"
+			(at 373.38 101.6 0)
+			(hide yes)
 			(show_name no)
 			(do_not_autoplace no)
@@
 			)
 		)
-		(property "Value" "S3B-XH-A-1(LF)(SN)"
-			(at 223.52 33.02 0)
+		(property "Value" "GND"
+			(at 373.38 100.33 0)
 			(show_name no)
 			(do_not_autoplace no)
@@
 			)
 		)
-		(property "Footprint" "Connector_JST:JST_XH_S3B-XH-A-1_1x03_P2.50mm_Horizontal"
-			(at 223.266 34.036 0)
+		(property "Footprint" ""
+			(at 373.38 95.25 0)
 			(hide yes)
 			(show_name no)
@@
 			(effects
 				(font
-					(size 0.5 0.5)
+					(size 1.27 1.27)
 				)
 			)
 		)
 		(property "Datasheet" ""
-			(at 223.52 39.37 0)
+			(at 373.38 95.25 0)
 			(hide yes)
 			(show_name no)
@@
 			)
 		)
-		(property "Description" ""
+		(property "Description" "Power symbol creates a global label with name \"GND\" , ground"
+			(at 373.38 95.25 0)
+			(hide yes)
+			(show_name no)
+			(do_not_autoplace no)
+			(effects
+				(font
+					(size 1.27 1.27)
+				)
+			)
+		)
+		(pin "1"
+		)
+		(instances
+			(project "saturn"
+				(path "/1437d78f-2672-4553-b786-22c28e887ed9"
+					(reference "#PWR035")
+					(unit 1)
+				)
+			)
+		)
+	)
+	(symbol
+		(lib_id "Connector_Generic_MountingPin:Conn_01x03_MountingPin")
+		(at 223.52 39.37 0)
+		(mirror x)
+		(unit 1)
+		(body_style 1)
+		(exclude_from_sim no)
+		(in_bom yes)
+		(on_board yes)
+		(in_pos_files yes)
+		(dnp no)
+		(fields_autoplaced yes)
+		(property "Reference" "J13"
+			(at 226.06 37.7443 0)
+			(show_name no)
+			(do_not_autoplace no)
+			(effects
+				(font
+					(size 1.27 1.27)
+				)
+				(justify left)
+			)
+		)
+		(property "Value" "ZX-XH2.54-3PWT"
+			(at 226.06 40.2843 0)
+			(show_name no)
+			(do_not_autoplace no)
+			(effects
+				(font
+					(size 1.27 1.27)
+				)
+				(justify left)
+			)
+		)
+		(property "Footprint" "JST-XH-SMT:JST-XH-SMD-3Pin"
 			(at 223.52 39.37 0)
 			(hide yes)
@@
 			)
 		)
-		(property "LCSC" "C163036"
+		(property "Datasheet" ""
 			(at 223.52 39.37 0)
 			(hide yes)
@@
 			)
 		)
-		(property "Basic/Extended" "E"
+		(property "Description" "Generic connectable mounting pin connector, single row, 01x03, script generated (kicad-library-utils/schlib/autogen/connector/)"
 			(at 223.52 39.37 0)
 			(hide yes)
@@
 			)
 		)
-		(property "JLCPCB_CORRECTION" "2.54;0;180"
+		(property "LCSC" "C7429672"
 			(at 223.52 39.37 0)
 			(hide yes)
@@
 			)
 		)
-		(property "Price (100ks)" "0.0675"
+		(property "Basic/Extended" "E"
 			(at 223.52 39.37 0)
 			(hide yes)
@@
 			)
 		)
-		(property "Price (1ks)" "0.0815"
+		(property "JLCPCB_CORRECTION" ""
 			(at 223.52 39.37 0)
 			(hide yes)
@@
 		(pin "3"
 		)
+		(pin "MP"
+		)
 		(instances
 			(project "saturn"
@@
 			)
 		)
-		(property "JLCPCB_CORRECTION" ""
+		(property "JLCPCB_CORRECTION" "0;0;-90"
 			(at 344.17 85.09 90)
 			(hide yes)
@@
 			)
 		)
-		(property "JLCPCB_CORRECTION" ""
+		(property "JLCPCB_CORRECTION" "0;0;-90"
 			(at 344.17 48.26 90)
 			(hide yes)
@@
 	)
 	(symbol
+		(lib_id "power:GND")
+		(at 394.97 177.8 0)
+		(unit 1)
+		(body_style 1)
+		(exclude_from_sim no)
+		(in_bom yes)
+		(on_board yes)
+		(in_pos_files yes)
+		(dnp no)
+		(property "Reference" "#PWR071"
+			(at 394.97 184.15 0)
+			(hide yes)
+			(show_name no)
+			(do_not_autoplace no)
+			(effects
+				(font
+					(size 1.27 1.27)
+				)
+			)
+		)
+		(property "Value" "GND"
+			(at 394.97 182.88 0)
+			(show_name no)
+			(do_not_autoplace no)
+			(effects
+				(font
+					(size 1.27 1.27)
+				)
+			)
+		)
+		(property "Footprint" ""
+			(at 394.97 177.8 0)
+			(hide yes)
+			(show_name no)
+			(do_not_autoplace no)
+			(effects
+				(font
+					(size 1.27 1.27)
+				)
+			)
+		)
+		(property "Datasheet" ""
+			(at 394.97 177.8 0)
+			(hide yes)
+			(show_name no)
+			(do_not_autoplace no)
+			(effects
+				(font
+					(size 1.27 1.27)
+				)
+			)
+		)
+		(property "Description" "Power symbol creates a global label with name \"GND\" , ground"
+			(at 394.97 177.8 0)
+			(hide yes)
+			(show_name no)
+			(do_not_autoplace no)
+			(effects
+				(font
+					(size 1.27 1.27)
+				)
+			)
+		)
+		(pin "1"
+		)
+		(instances
+			(project "saturn"
+				(path "/1437d78f-2672-4553-b786-22c28e887ed9"
+					(reference "#PWR071")
+					(unit 1)
+				)
+			)
+		)
+	)
+	(symbol
 		(lib_id "Switch:SW_Push")
 		(at 33.02 208.28 0)
@@
 	)
 	(symbol
-		(lib_id "Connector_Generic:Conn_01x10")
+		(lib_id "Connector_Generic_MountingPin:Conn_01x10_MountingPin")
 		(at 389.89 200.66 0)
 		(mirror x)
@@
 		(dnp no)
 		(property "Reference" "J6"
-			(at 392.43 200.6601 0)
+			(at 389.128 214.884 0)
 			(show_name no)
 			(do_not_autoplace no)
@@
 			)
 		)
-		(property "Value" "Conn_01x10"
-			(at 392.43 198.1201 0)
+		(property "Value" "ZX-XH2.54-10PWT"
+			(at 383.286 218.44 0)
 			(show_name no)
 			(do_not_autoplace no)
@@
 			)
 		)
-		(property "Footprint" "Connector_JST:JST_XH_S10B-XH-A-1_1x10_P2.50mm_Horizontal"
+		(property "Footprint" "JST-XH-SMT:JST-XH-SMD-10Pin"
 			(at 389.89 200.66 0)
 			(hide yes)
@@
 			)
 		)
-		(property "Description" "Generic connector, single row, 01x10, script generated (kicad-library-utils/schlib/autogen/connector/)"
+		(property "Description" "Generic connectable mounting pin connector, single row, 01x10, script generated (kicad-library-utils/schlib/autogen/connector/)"
 			(at 389.89 200.66 0)
 			(hide yes)
@@
 			)
 		)
-		(property "LCSC" "C491718"
+		(property "LCSC" "C7429679"
 			(at 389.89 200.66 0)
 			(hide yes)
@@
 			)
 		)
-		(property "JLCPCB_CORRECTION" "11.25;0;0"
+		(property "JLCPCB_CORRECTION" ""
 			(at 389.89 200.66 0)
 			(hide yes)
@@
 		(pin "8"
 		)
+		(pin "MP"
+		)
 		(instances
 			(project "saturn"
@@
 			)
 		)
-		(property "JLCPCB_CORRECTION" ""
+		(property "JLCPCB_CORRECTION" "0;0;-90"
 			(at 262.89 48.26 90)
 			(hide yes)

Commit message: Tune silkscreen, enlarge SMT switch pads
Parts:
- SW2, SW3: footprint Button_Switch_SMD:SW_Push_1P1T_NO_Vertical_Wuerth_434133025816 -> Switch_SMT:SW_SMD_LargePads
Changed lines of the file:
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@@
 			)
 		)
-		(property "Footprint" "Button_Switch_SMD:SW_Push_1P1T_NO_Vertical_Wuerth_434133025816"
+		(property "Footprint" "Switch_SMT:SW_SMD_LargePads"
 			(at 33.02 203.2 0)
 			(hide yes)
@@
 			)
 		)
-		(property "Footprint" "Button_Switch_SMD:SW_Push_1P1T_NO_Vertical_Wuerth_434133025816"
+		(property "Footprint" "Switch_SMT:SW_SMD_LargePads"
 			(at 33.02 165.1 0)
 			(hide yes)

Commit message: Use 0805 10u capacitors (cheaper)
Parts:
- C1, C24, C3, C4, C5, C6: footprint Capacitor_SMD:C_1206_3216Metric -> Capacitor_SMD:C_0805_2012Metric; LCSC C13585 -> C15850
- J11: footprint Connector_USB:USB_Micro-B_Molex-105017-0001 -> USB_Conn:USB_Micro-B_XNJ-073_With_THR_Paste
- J12: footprint Connector_USB:USB_C_Receptacle_HRO_TYPE-C-31-M-12 -> USB_Conn:USB_C_Receptacle_HRO_TYPE-C-31-M-12_With_THR_Paste; Price (100ks) 0.1238 -> (none); Price (1ks) 0.1542 -> (none)
- U1: footprint RKL-ESP:ESP32-S3-WROOM -> ESP32-WROOM:ESP32-S3-WROOM
- U9: footprint LED_SMD:LED_WS2812B-2020_PLCC4_2.0x2.0mm -> XL-2020RGBC-WS2812B:LED_WS2812B-2020_PLCC4_2.0x2.0mm
Changed lines of the file:
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@@
 			)
 		)
-		(property "Footprint" "Capacitor_SMD:C_1206_3216Metric"
+		(property "Footprint" "Capacitor_SMD:C_0805_2012Metric"
 			(at 211.7852 95.25 0)
 			(hide yes)
@@
 			)
 		)
-		(property "LCSC" "C13585"
+		(property "LCSC" "C15850"
 			(at 210.82 91.44 0)
 			(hide yes)
@@
 			)
 		)
-		(property "Footprint" "Connector_USB:USB_Micro-B_Molex-105017-0001"
+		(property "Footprint" "USB_Conn:USB_Micro-B_XNJ-073_With_THR_Paste"
 			(at 33.02 101.6 0)
 			(hide yes)
@@
 			)
 		)
-		(property "Footprint" "Capacitor_SMD:C_1206_3216Metric"
+		(property "Footprint" "Capacitor_SMD:C_0805_2012Metric"
 			(at 58.1152 256.54 0)
 			(hide yes)
@@
 			)
 		)
-		(property "LCSC" "C13585"
+		(property "LCSC" "C15850"
 			(at 57.15 252.73 0)
 			(hide yes)
@@
 			)
 		)
-		(property "Footprint" "LED_SMD:LED_WS2812B-2020_PLCC4_2.0x2.0mm"
+		(property "Footprint" "XL-2020RGBC-WS2812B:LED_WS2812B-2020_PLCC4_2.0x2.0mm"
 			(at 176.53 22.86 0)
 			(hide yes)
@@
 			)
 		)
-		(property "Footprint" "Capacitor_SMD:C_1206_3216Metric"
+		(property "Footprint" "Capacitor_SMD:C_0805_2012Metric"
 			(at 126.0602 40.64 0)
 			(hide yes)
@@
 			)
 		)
-		(property "LCSC" "C13585"
+		(property "LCSC" "C15850"
 			(at 125.095 36.83 0)
 			(hide yes)
@@
 			)
 		)
-		(property "Footprint" "RKL-ESP:ESP32-S3-WROOM"
+		(property "Footprint" "ESP32-WROOM:ESP32-S3-WROOM"
 			(at 256.54 87.63 0)
 			(hide yes)
@@
 			)
 		)
-		(property "Footprint" "Capacitor_SMD:C_1206_3216Metric"
+		(property "Footprint" "Capacitor_SMD:C_0805_2012Metric"
 			(at 67.0052 121.92 0)
 			(hide yes)
@@
 			)
 		)
-		(property "LCSC" "C13585"
+		(property "LCSC" "C15850"
 			(at 66.04 118.11 0)
 			(hide yes)
@@
 			)
 		)
-		(property "Footprint" "Connector_USB:USB_C_Receptacle_HRO_TYPE-C-31-M-12"
+		(property "Footprint" "USB_Conn:USB_C_Receptacle_HRO_TYPE-C-31-M-12_With_THR_Paste"
 			(at 33.655 44.45 0)
 			(hide yes)
@@
 			)
 		)
-		(property "Datasheet" "https://www.usb.org/sites/default/files/documents/usb_type-c.zip"
+		(property "Datasheet" ""
 			(at 33.655 44.45 0)
 			(hide yes)
@@
 			)
 		)
-		(property "Price (100ks)" "0.1238"
-			(at 29.845 44.45 0)
-			(hide yes)
-			(show_name no)
-			(do_not_autoplace no)
-			(effects
-				(font
-					(size 1.27 1.27)
-				)
-			)
-		)
-		(property "Price (1ks)" "0.1542"
-			(at 29.845 44.45 0)
-			(hide yes)
-			(show_name no)
-			(do_not_autoplace no)
-			(effects
-				(font
-					(size 1.27 1.27)
-				)
-			)
-		)
 		(pin "A1"
 		)
@@
 			)
 		)
-		(property "Footprint" "Capacitor_SMD:C_1206_3216Metric"
+		(property "Footprint" "Capacitor_SMD:C_0805_2012Metric"
 			(at 35.2552 256.54 0)
 			(hide yes)
@@
 			)
 		)
-		(property "LCSC" "C13585"
+		(property "LCSC" "C15850"
 			(at 34.29 252.73 0)
 			(hide yes)
@@
 			)
 		)
-		(property "Footprint" "Capacitor_SMD:C_1206_3216Metric"
+		(property "Footprint" "Capacitor_SMD:C_0805_2012Metric"
 			(at 340.0552 227.33 0)
 			(hide yes)
@@
 			)
 		)
-		(property "LCSC" "C13585"
+		(property "LCSC" "C15850"
 			(at 339.09 223.52 0)
 			(hide yes)
